File: Vessel.kicad_pcb (KiCad board)
At the start: 2 copper layers, 338.6 x 174.3 mm, 219 parts, among them SW1 SW_PUSH, U1 ATMEGA32U4, X1 XTAL_GND

Commit message: Routing Done - Via lowered
Routing:
- net /row5: track 0.00 -> 494.7 mm, vias 0 -> 1
- net /col3: track 0.00 -> 483.4 mm
- net /col0: track 0.00 -> 478.1 mm
- net /row4: track 0.00 -> 467.8 mm, vias 0 -> 2
- net /row6: track 0.00 -> 464.4 mm, vias 0 -> 1
- net /col1: track 0.00 -> 445.0 mm, vias 0 -> 1
- net /row3: track 0.00 -> 439.2 mm, vias 0 -> 1
- net /row2: track 0.00 -> 436.3 mm, vias 0 -> 1
- net /col2: track 0.00 -> 416.6 mm, vias 0 -> 2
- net /row1: track 0.00 -> 409.9 mm, vias 0 -> 1
- net /row0: track 0.00 -> 395.6 mm, vias 0 -> 1
- net /col4: track 0.00 -> 369.4 mm, vias 0 -> 1
- net /col6: track 0.00 -> 367.4 mm
- net /col5: track 0.00 -> 365.2 mm
- net /col7: track 0.00 -> 313.0 mm
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- added copper zone on F.Cu, net GND
- removed copper zone on B.Cu, net GND
- removed copper zone on F.Cu, net VCC
Other:
- net class Default removed
